File: Inputs_out_Puts.kicad_sch (KiCad schematic)
At the start: 37 parts, among them J1 Conn_01x03_Pin, J14 USB_C_Receptacle_USB2.0, J4 Conn_01x02_Female, J8 Conn_01x03_MountingPin, J9 Conn_01x06_MountingPin, SW1 SW_MEC_5G, U1 TCAN330, U2 TPS709-5

Commit message: attempt at cleaning up
Parts:
- removed C14: 1uF, Capacitor_SMD:C_0603_1608Metric, symbol Device:C
- removed C15: 100nF, Capacitor_SMD:C_0603_1608Metric, symbol Device:C
- removed C20: 2.2uf, Capacitor_SMD:C_1206_3216Metric, symbol Device:C
- removed C31: 220uF, Capacitor_SMD:CP_Elec_8x10, symbol Device:CP
- removed D6: LED, LED_SMD:LED_0805_2012Metric, symbol Device:LED
- removed J9: Conn_01x06_MountingPin, Connector_JST:JST_SH_BM06B-SRSS-TB_1x06-1MP_P1.00mm_Vertical, symbol Connector_Generic_MountingPin:Conn_01x06_MountingPin
- removed JP1: Jumper_3_Bridged12, Jumper:SolderJumper-3_P1.3mm_Bridged2Bar12_RoundedPad1.0x1.5mm_NumberLabels, symbol Jumper:Jumper_3_Bridged12
- removed R7: 220, Resistor_SMD:R_0603_1608Metric, symbol Device:R
- removed SW1: SW_MEC_5G, mystuff:SW_SPST_TS-1187A-B, symbol Switch:SW_Push
- removed TP10: TestPoint, TestPoint:TestPoint_Pad_D1.5mm, symbol Connector:TestPoint
- removed TP7, TP8, TP9: TestPoint, TestPoint:TestPoint_Pad_D1.0mm, symbol Connector:TestPoint
- removed U1: TCAN330, Package_SO:SOIC-8_3.9x4.9mm_P1.27mm, symbol Interface_CAN_LIN:TCAN330
- removed U2: TPS709-5, Package_TO_SOT_SMD:TSOT-23-5, symbol mystuff:TPS709-5
- added C3: 2.2uf, Capacitor_SMD:C_1206_3216Metric, symbol Device:C
- added D4_white2: LED, LED_SMD:LED_0805_2012Metric, symbol Device:LED
- added J2: Conn_01x12_MountingPin, mystuff:0.5K-A-12PBF, symbol Connector_Generic_MountingPin:Conn_01x12_MountingPin
- added J5: Conn_01x03_MountingPin, Connector_JST:JST_SH_BM03B-SRSS-TB_1x03-1MP_P1.00mm_Vertical, symbol Connector_Generic_MountingPin:Conn_01x03_MountingPin
- added J6: Conn_01x06_MountingPin, Connector_PinHeader_1.27mm:PinHeader_1x06_P1.27mm_Vertical, symbol Connector_Generic_MountingPin:Conn_01x06_MountingPin
- added JP4: Jumper_2_Bridged, Jumper:SolderJumper-2_P1.3mm_Bridged_RoundedPad1.0x1.5mm, symbol Jumper:Jumper_2_Bridged
- added U2: TJA1057T/1Z, Package_SO:SOIC-8_3.9x4.9mm_P1.27mm, symbol Interface_CAN_LIN:TJA1051T
- C41: footprint Capacitor_SMD:C_0603_1608Metric -> Capacitor_SMD:C_0402_1005Metric
- H1, H2, H3, H4: footprint MountingHole:MountingHole_3.2mm_M3_ISO14580 -> MountingHole:MountingHole_2.2mm_M2
- J1: footprint mystuff:flat_3 -> Connector_JST:JST_XH_B3B-XH-AM_1x03_P2.50mm_Vertical
- J4: footprint Connector_AMASS:AMASS_XT30PW-M_1x02_P2.50mm_Horizontal -> Connector_PinHeader_2.54mm:PinHeader_1x02_P2.54mm_Vertical
- R19: footprint Resistor_SMD:R_0603_1608Metric -> Resistor_SMD:R_0402_1005Metric; LCSC Part C23186 -> (none)
- R20, R5, R6, R98: footprint Resistor_SMD:R_0603_1608Metric -> Resistor_SMD:R_0402_1005Metric
- R8: value 100k -> 220; footprint Resistor_SMD:R_0603_1608Metric -> Resistor_SMD:R_0402_1005Metric
- R99: value 10k -> 10K; footprint Resistor_SMD:R_0603_1608Metric -> Resistor_SMD:R_0402_1005Metric
- renumbered D4 to D4_white1
Connections:
- net nRST is gone; now on net GND: R8.2
- net CAN_SHDN: now also R99.1; no longer R99.2
- net FDCAN1_RX/BOOT_0: now also U2.4 (RXD)
- net FDCAN1_TX: now also U2.1 (TXD)
- net GND: now also C3.2, J2.10 (Pin_10), J2.11 (Pin_11), J2.8 (Pin_8), J2.MP (MountPin), J5.3 (Pin_3), J5.MP (MountPin), J6.2 (Pin_2), J6.MP (MountPin), U2.2 (GND)
- net GPIO_PA10: now also J2.5 (Pin_5)
- net I2C2_SCL: now also J2.7 (Pin_7)
- net I2C2_SDA: now also J2.6 (Pin_6)
- net SPI1_MISO: now also J2.3 (Pin_3)
- net SPI1_MOSI: now also J2.2 (Pin_2)
- net SPI1_NSS: now also J2.4 (Pin_4)
- net SPI1_SCK: now also J2.1 (Pin_1)
- net USER2: now also D4_white2.2 (A)
- net VDD: now also J6.3 (Pin_3), U2.3 (VCC); no longer R8.1
- net VM: now also C3.1, J2.12 (Pin_12)
- net at J8.1 (Pin_1): now also J5.1 (Pin_1), JP4.2 (B), U2.6 (CANL); no longer R98.2
- net at R98.1: now also JP4.1 (A); no longer J8.2 (Pin_2)
- new net: D4_white2.1 (K), R8.1
- new net: R99.2, U2.8 (S)
- new net CAN_Termination: J5.2 (Pin_2), J8.2 (Pin_2), R98.2, U2.7 (CANH)
- new net HA: J6.4 (Pin_4)
- new net HB: J6.5 (Pin_5)
- new net HC: J6.6 (Pin_6)
- new net Thermistor: J6.1 (Pin_1)
Other:
- note removed: "Actually TPS709?"
- moved on the sheet: J4, R98
