File: Power_Stage.kicad_sch (KiCad schematic)
At the start: 25 parts, among them Q1 Q_NMOS_GDS, Q2 Q_NMOS_GDS, Q3 Q_NMOS_GDS, Q4 Q_NMOS_GDS, Q5 Q_NMOS_GDS, Q6 Q_NMOS_GDS

Commit message: attempt at cleaning up
Parts:
- removed Q1, Q2, Q3, Q4, Q5, Q6: Q_NMOS_GDS, my_stuff:DFN-8-1EP_6x5mm_P1.27mm_EP4x4mm, symbol Device:Q_NMOS_GDS
- removed R10: 4mΩ, Resistor_SMD:R_2512_6332Metric, symbol MotorController:TAYLOR_RESISTOR
- added Q1, Q2, Q7: Q_Dual_NMOS_G1, mystuff:V-DFN3030-8 (Type K), symbol mystuff:Q_Dual_NMOS_G1
- added R7: 7mΩ, Resistor_SMD:R_1206_3216Metric, symbol MotorController:TAYLOR_RESISTOR
- R1, R13, R17, R18, R25, R4: footprint Resistor_SMD:R_0603_1608Metric -> Resistor_SMD:R_0402_1005Metric; LCSC Part C23140 -> (none)
- R15: value 4mΩ -> 7mΩ; footprint Resistor_SMD:R_2512_6332Metric -> Resistor_SMD:R_1206_3216Metric; LCSC C375693 -> C76302
Connections:
- net GND: now also Q7.S2, R7.1
- net OUT1: now also Q7.S1/D2
- net OUT2: now also Q1.S1/D2
- net OUT3: now also Q2.S1/D2
- net VM: now also Q1.D1 (D), Q2.D1 (D), Q7.D1 (D)
- net VSHUNT1P: now also Q2.S2, R7.2
- net VSHUNT2P: now also Q1.S2
- net at D7.2 (A), R13.1: now also Q7.G1
- net at D2.2 (A), R25.1: now also Q7.G2
- net at D12.2 (A), R18.1: now also Q2.G2
- net at D1.2 (A), R1.1: now also Q1.G1
- net at D10.2 (A), R4.1: now also Q1.G2
- net at D11.2 (A), R17.1: now also Q2.G1
Other:
- note removed: "Have removed jumpers for space"
- note removed: "Replace jumper with pass throuhg"
- moved on the sheet: C16, C24, C27, D1, D10, D11, D12, D2, D7, NT1, NT2, R1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
