File: STSPIN32G4_V2.kicad_sch (KiCad schematic)
At the start: 32 parts, among them IC1 STSPIN32G4, J1 Conn_01x02_Male, J2 Conn_01x06_Male, J7 Conn_01x02, U3 AS5045B, Y3 24mhz

Commit message: attempt at cleaning up
Parts:
- removed C12: 100nF, Capacitor_SMD:C_0603_1608Metric, symbol Device:C
- removed C14: 0.1uF, Capacitor_SMD:C_0603_1608Metric_Pad1.08x0.95mm_HandSolder, symbol Device:C
- removed C3: N.M., Capacitor_SMD:C_0603_1608Metric, symbol Device:C
- removed J1: Conn_01x02_Male, Connector_PinSocket_2.54mm:PinSocket_1x02_P2.54mm_Vertical, symbol Connector:Conn_01x02_Male
- removed J2: Conn_01x06_Male, Connector_PinSocket_2.54mm:PinSocket_1x06_P2.54mm_Vertical, symbol Connector:Conn_01x06_Male
- removed J7: Conn_01x02, Connector_PinHeader_2.54mm:PinHeader_1x02_P2.54mm_Vertical, symbol Connector_Generic:Conn_01x02
- removed JP1, JP2: Jumper_2_Bridged, Jumper:SolderJumper-2_P1.3mm_Bridged_RoundedPad1.0x1.5mm, symbol Jumper:Jumper_2_Bridged
- removed JP3: Jumper_NC_Dual, Jumper:SolderJumper-3_P1.3mm_Open_RoundedPad1.0x1.5mm_NumberLabels, symbol Device:Jumper_NC_Dual
- removed TP3, TP4, TP5, TP6: TestPoint, TestPoint:TestPoint_Pad_D1.0mm, symbol Connector:TestPoint
- removed U3: AS5045B, Package_SO:SSOP-16_5.3x6.2mm_P0.65mm, symbol Sensor_Magnetic:AS5045B
- added J9: Conn_01x06_MountingPin, Connector_JST:JST_SH_BM06B-SRSS-TB_1x06-1MP_P1.00mm_Vertical, symbol Connector_Generic_MountingPin:Conn_01x06_MountingPin
- added JP3: Jumper_2_Open, Jumper:SolderJumper-2_P1.3mm_Open_TrianglePad1.0x1.5mm, symbol Jumper:Jumper_2_Open
- added R11: 10k, Resistor_SMD:R_0402_1005Metric, symbol Device:R
- added SW1: SW_Push, Jumper:SolderJumper-2_P1.3mm_Open_RoundedPad1.0x1.5mm, symbol Switch:SW_Push
- C10, C8: footprint Capacitor_SMD:C_0603_1608Metric -> Capacitor_SMD:C_0402_1005Metric; LCSC Part C15849 -> (none)
- C11, C7, C9: footprint Capacitor_SMD:C_0603_1608Metric -> Capacitor_SMD:C_0402_1005Metric; LCSC Part C14663 -> (none)
- C18: footprint Capacitor_SMD:C_0603_1608Metric -> Capacitor_SMD:C_0402_1005Metric; LCSC C1648 -> (none)
- C4: renamed from C1; footprint Capacitor_SMD:C_0603_1608Metric -> Capacitor_SMD:C_0402_1005Metric; LCSC C1648 -> (none)
- D5: footprint Diode_SMD:D_SMA -> Diode_SMD:D_SOD-323; LCSC C14996 -> C191023
- IC1: LCSC (none) -> C2858620
- L2: footprint Inductor_SMD:L_Bourns-SRN6028 -> Inductor_SMD:L_1812_4532Metric; LCSC C467143 -> C394124
- R2: value 22k -> 10k; footprint Resistor_SMD:R_0603_1608Metric -> Resistor_SMD:R_0402_1005Metric; LCSC Part C31850 -> (none)
- R3: footprint Resistor_SMD:R_0603_1608Metric -> Resistor_SMD:R_0402_1005Metric; LCSC Part C25804 -> (none)
- renumbered C$1 to C1
Connections:
- net HALL2 is gone; now on net CAN_SHDN: IC1.58 (PB7)
- net VBAT is gone; now on net VDD: IC1.2 (VBAT)
- net VDDA is gone; now on net VDD: C8.1, C9.1, IC1.27 (VDDA)
- net VREGIN is gone; now on net VCC: IC1.64 (REGIN)
- net CAN_SHDN: no longer IC1.4 (PC14)
- net GND: now also J9.4 (Pin_4), J9.MP (MountPin), R11.2
- net OPN3: no longer IC1.25 (PB2)
- net OPO3: no longer IC1.24 (PB1)
- net OPP3: no longer IC1.23 (PB0)
- net SCREF: now also JP3.1 (A)
- net SPI1_SCK: now also J9.1 (Pin_1)
- net SWCLK: now also J9.5 (Pin_5)
- net SWDIO: now also J9.3 (Pin_3)
- net VDD: now also J9.6 (Pin_6), JP3.2 (B), SW1.2
- net nRST: now also J9.2 (Pin_2)
- net HB: now reaches IC1.12 (PC3)
- net I2C2_SDA: now reaches IC1.44 (PA8)
- net PC15: now reaches IC1.5 (PC15)
- net CAN_RX renamed D-
- net CAN_TX renamed D+
- net HALL1: no longer names the net of IC1.57 (PB6)
- net HALL3 renamed FDCAN1_RX/BOOT_0
- net FDCAN1_RX/BOOT_0: now also R11.1, SW1.1
- net I2C1_SCL: no longer names the net of IC1.51 (PA15)
- net I2C1_SDA renamed FDCAN1_TX
- net UART_RX renamed GPIO_PA10
- net UART_TX renamed I2C2_SCL
- net VBUS renamed VBUS_Monitor
- net VOUT1 renamed HA
- net VOUT2 renamed Thermistor
- net VOUT3 renamed HC
Other:
- note added: "ENC_A"
- note added: "ENC_B"
- note added: "ENC_I"
- note added: "These caps (C8,C9) for VDA"
- note removed: "Can likely remove some of these jumpers"
- note removed: "PAD is disconnected need to connect with solder!"
